File: hardware/Air-Sus/LEDs.kicad_sch (KiCad schematic)
At the start: 10 parts

Commit message: air-sus layout check e Please enter the commit message for your changes. Lines starting
Changed lines of the file:
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@@
 	(text_box "LED\n"
 		(exclude_from_sim no)
-		(at 115.57 62.23 0)
+		(at 116.84 113.03 0)
 		(size 66.04 46.99)
 		(margins 0.9525 0.9525 0.9525 0.9525)

Commit message: finished rev a layout for all 3 boards + added cubemx file
Parts:
- R14, R15, R16, R17, R18: P/N C21190 -> CRCW06031K00FKEI
Connections:
- net diff_status renamed Diff_Status
Changed lines of the file:
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@@
 	(text_box "LED\n"
 		(exclude_from_sim no)
-		(at 116.84 113.03 0)
+		(at 115.57 62.23 0)
 		(size 66.04 46.99)
 		(margins 0.9525 0.9525 0.9525 0.9525)
@@
 	(wire
 		(pts
-			(xy 147.32 78.74) (xy 147.32 81.28)
+			(xy 147.32 77.47) (xy 147.32 81.28)
 		)
 		(stroke
@@
 	(wire
 		(pts
-			(xy 157.48 78.74) (xy 157.48 81.28)
+			(xy 157.48 77.47) (xy 157.48 81.28)
 		)
 		(stroke
@@
 	(wire
 		(pts
-			(xy 167.64 78.74) (xy 167.64 81.28)
+			(xy 167.64 77.47) (xy 167.64 81.28)
 		)
 		(stroke
@@
 		)
 	)
-	(global_label "diff_status"
+	(hierarchical_label "Diff_Status"
 		(shape input)
-		(at 147.32 78.74 90)
-		(fields_autoplaced yes)
+		(at 147.32 77.47 90)
 		(effects
 			(font
@@
 			(justify left)
 		)
-		(property "Intersheetrefs" "${INTERSHEET_REFS}"
-			(at 147.32 65.7764 90)
-			(effects
-				(font
-					(size 1.27 1.27)
-				)
-				(justify left)
-				(hide yes)
-			)
-		)
-	)
-	(global_label "ir_status"
+	)
+	(hierarchical_label "Temp_status"
 		(shape input)
-		(at 157.48 78.74 90)
-		(fields_autoplaced yes)
+		(at 167.64 77.47 90)
 		(effects
 			(font
@@
 			(justify left)
 		)
-		(property "Intersheetrefs" "${INTERSHEET_REFS}"
-			(at 157.48 67.5906 90)
-			(effects
-				(font
-					(size 1.27 1.27)
-				)
-				(justify left)
-				(hide yes)
-			)
-		)
-	)
-	(global_label "Temp_status"
+	)
+	(hierarchical_label "ir_status"
 		(shape input)
-		(at 167.64 78.74 90)
-		(fields_autoplaced yes)
+		(at 157.48 77.47 90)
 		(effects
 			(font
@@
 			(justify left)
 		)
-		(property "Intersheetrefs" "${INTERSHEET_REFS}"
-			(at 167.64 64.0831 90)
-			(effects
-				(font
-					(size 1.27 1.27)
-				)
-				(justify left)
-				(hide yes)
-			)
-		)
 	)
 	(symbol
@@
 			)
 		)
-		(property "P/N" "C21190"
+		(property "P/N" "CRCW06031K00FKEI "
 			(at 157.48 85.09 0)
 			(effects
@@
 			)
 		)
-		(property "P/N" "C21190"
+		(property "P/N" "CRCW06031K00FKEI "
 			(at 135.89 85.09 0)
 			(effects
@@
 			)
 		)
-		(property "P/N" "C21190"
+		(property "P/N" "CRCW06031K00FKEI "
 			(at 167.64 85.09 0)
 			(effects
@@
 			)
 		)
-		(property "P/N" "C21190"
+		(property "P/N" "CRCW06031K00FKEI "
 			(at 123.19 85.09 0)
 			(effects
@@
 			)
 		)
-		(property "P/N" "C21190"
+		(property "P/N" "CRCW06031K00FKEI "
 			(at 147.32 85.09 0)
 			(effects
