File: hardware/Air-Sus/Air-Sus.kicad_pcb (KiCad board)
At the start: 2 copper layers, 50.1 x 63.6 mm, 54 parts, among them IC1 ABPMRRV060MG2A3, IC3 ABPMRRV060MG2A3, J1 53307-2471, J2 Conn_01x05, J4 MX150_02x06_Vertical, J5 Conn_01x06, U1 Opamp_Dual, U2 LDO40LPURY

Commit message: relayout
Parts:
- removed C7: 0.1uF, Capacitor_SMD:C_0603_1608Metric_Pad1.08x0.95mm_HandSolder
- removed G***: LOGO, UTSVT_Logos:UTSVT_Logo_Symbol
- removed G***: LHRs_LOGO, UTSVT_Logos:LHRs_LOGO
- removed U1: Opamp_Dual, TLV900QDRQ1:SOIC8_D_TEX
- added C10: 0.1uF, Capacitor_SMD:C_0603_1608Metric_Pad1.08x0.95mm_HandSolder, F.Cu at (-22.6, -24.7)
- added U3: TLV9002QDRQ1, Air-Sus Footprints:SOIC8_D_TEX, F.Cu at (-20.5, -29.3)
- 24v_TP1, 3.3v_TP1, GNDA_TP1, GNDA_TP2, GND_TP1, GND_TP2, GND_TP3, LinPot_TP1, PressureErr_TP1, PressureErr_TP2, VDDA_TP1: moved to F.Cu
- IC1, IC3: footprint footprints:ABPMRRV060MG2A3 -> Air-Sus Footprints:ABPMRRV060MG2A3
- RN1, RN2, RN4, RN5, RN6, RN7: footprint 4pinRes:YC324JK07220RL -> Air-Sus Footprints:YC324JK07220RL
- moved RN7 178.5 mm to (218.6, -68.0), turned to -90 degrees
- moved RN2 177.4 mm to (209.5, -68.0), turned to 90 degrees
- moved RN6 176.8 mm to (218.6, -60.0), turned to -90 degrees
- moved RN5 175.7 mm to (209.5, -60.0), turned to 90 degrees
- moved J4 174.7 mm to (205.2, -77.1)
- moved RN1 160.6 mm to (218.6, -52.0), turned to -90 degrees
- moved RN4 159.3 mm to (209.5, -52.0), turned to 90 degrees
- moved J1 151.7 mm to (143.3, -103.0)
- moved D10 126.2 mm to (17.7, 28.2), turned to 0 degrees
- moved D9 126.1 mm to (17.7, 25.6), turned to 0 degrees
- moved D7 125.9 mm to (17.7, 20.6), turned to 0 degrees
- moved D8 125.9 mm to (17.7, 23.1), turned to 0 degrees
- moved D3 125.9 mm to (17.7, 18.1), turned to 0 degrees
- moved J2 121.2 mm to (28.5, 27.4)
- moved R18 120.0 mm to (17.7, 40.7)
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Connections:
- RN1 pad 1: /mx150Connector/Gen_5 -> /mx150Connector/Gen_8
- RN1 pad 2: /mx150Connector/Gen_6 -> /mx150Connector/Gen_7
- RN1 pad 3: /mx150Connector/Gen_7 -> /mx150Connector/Gen_6
- RN1 pad 4: /mx150Connector/Gen_8 -> /mx150Connector/Gen_5
- RN1 pad 5: /SCL2 -> +3.3V
- RN1 pad 6: GND -> /SDA2
- RN1 pad 7: /SDA2 -> GND
- RN1 pad 8: +3.3V -> /SCL2
- RN5 pad 1: /mx150Connector/Gen_1 -> /mx150Connector/Gen_4
- RN5 pad 2: /mx150Connector/Gen_2 -> /mx150Connector/Gen_3
- RN5 pad 3: /mx150Connector/Gen_3 -> /mx150Connector/Gen_2
- RN5 pad 4: /mx150Connector/Gen_4 -> /mx150Connector/Gen_1
- RN5 pad 5: GND -> +24V
- RN5 pad 6: /CAN_L -> /CAN_H
- RN5 pad 7: /CAN_H -> /CAN_L
- RN5 pad 8: +24V -> GND
- RN7 pad 1: /mx150Connector/Gen_5 -> /mx150Connector/Gen_8
- RN7 pad 2: /mx150Connector/Gen_6 -> /mx150Connector/Gen_7
- RN7 pad 3: /mx150Connector/Gen_7 -> /mx150Connector/Gen_6
- RN7 pad 4: /mx150Connector/Gen_8 -> /mx150Connector/Gen_5
- RN7 pad 5: /CAN_L -> +24V
- RN7 pad 6: GND -> /CAN_H
- RN7 pad 7: /CAN_H -> GND
- RN7 pad 8: +24V -> /CAN_L
Routing:
- net GND: track 164.6 -> 17.4 mm, vias 31 -> 0
- net /SDA: track 140.4 -> 0.00 mm, vias 15 -> 0
- net /SCL: track 135.0 -> 0.00 mm, vias 14 -> 0
- net /SDA2: track 100.4 -> 0.00 mm, vias 7 -> 0
- net /SCL2: track 97.8 -> 0.00 mm, vias 9 -> 0
- net /pressure_err2: track 74.0 -> 0.00 mm, vias 6 -> 0
- net +24V: track 77.7 -> 5.10 mm, vias 9 -> 1
- net +3.3V MCU: track 72.2 -> 0.00 mm, vias 8 -> 0
- net GNDA: track 64.5 -> 0.00 mm, vias 7 -> 0
- net /pressure_err1: track 56.4 -> 0.00 mm, vias 4 -> 0
- net +3.3V: track 45.4 -> 0.00 mm, vias 15 -> 0
- net linpot_out: track 44.0 -> 0.00 mm, vias 6 -> 0
- net /Temp_status: track 29.7 -> 0.00 mm, vias 2 -> 0
- net /IR_INTER: track 28.1 -> 0.00 mm, vias 2 -> 0
- net Net-(U2-Vout): track 26.3 -> 0.00 mm, vias 2 -> 0
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- removed copper zone on F.Cu, net +3.3V
- removed copper zone on B.Cu, net GND
Other:
- board outline removed
