File: hardware/Air-Sus/diffpress.kicad_sch (KiCad schematic)
At the start: 6 parts, among them IC1 ABPMRRV060MG2A3

Commit message: relayout
Parts:
- IC1: footprint footprints:ABPMRRV060MG2A3 -> Air-Sus Footprints:ABPMRRV060MG2A3
Changed lines of the file:
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@@
 			)
 		)
-		(property "Footprint" "footprints:ABPMRRV060MG2A3"
+		(property "Footprint" "Air-Sus Footprints:ABPMRRV060MG2A3"
 			(at 124.46 -25.07 0)
 			(effects
