File: hardware/Air-Sus/mx150Connector.kicad_sch (KiCad schematic)
At the start: 25 parts, among them J4 MX150_02x06_Vertical

Commit message: air-sus layout check e Please enter the commit message for your changes. Lines starting
Parts:
- removed R10, R11, R19, R20, R21, R22, R23, R24, R25, R26, R27, R28, R29, R30, R31, R32, R33, R34, R35, R36, R37, R6, R7, R8: 0, Resistor_SMD:R_0603_1608Metric_Pad0.98x0.95mm_HandSolder, symbol Device:R
- added RN1, RN2, RN4, RN5, RN6, RN7: YC324-JK-070RL, 4pinRes:YC324JK07220RL, symbol 4PinConn:YC324-JK-070RL
Connections:
- net +24V: now also RN2.8, RN5.8, RN7.8
- net +3.3V: now also RN1.8, RN4.8, RN6.8
- net CAN_H: now also RN2.7, RN5.7, RN7.7
- net CAN_L: now also RN2.6, RN5.6, RN7.5
- net GND: now also RN1.6, RN2.5, RN4.5, RN5.5, RN7.6
- net GNDA: now also RN6.6
- net Gen_1: now also RN2.1, RN4.1, RN5.1
- net Gen_2: now also RN2.2, RN4.2, RN5.2
- net Gen_3: now also RN2.3, RN4.3, RN5.3
- net Gen_4: now also RN2.4, RN4.4, RN5.4
- net Gen_5: now also RN1.1, RN6.1, RN7.1
- net Gen_6: now also RN1.2, RN6.2, RN7.2
- net Gen_7: now also RN1.3, RN6.3, RN7.3
- net Gen_8: now also RN1.4, RN6.4, RN7.4
- net SCL2: now also RN1.7, RN4.7
- net SDA2: now also RN1.5, RN4.6
- net linpot_out: now also RN6.7

Commit message: finished rev a layout for all 3 boards + added cubemx file
Parts:
- RN1, RN2, RN4, RN5, RN6, RN7: P/N (none) -> 603-YC324-JK-070RL
Connections:
- net SCL2: no longer RN4.7
- net SDA2: no longer RN4.6
- new net SCL: RN4.7
- new net SDA: RN4.6
Changed lines of the file:
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@@
 		)
 	)
-	(global_label "CAN_H"
-		(shape input)
+	(hierarchical_label "CAN_H"
+		(shape bidirectional)
 		(at 198.12 82.55 0)
-		(fields_autoplaced yes)
 		(effects
 			(font
@@
 			(justify left)
 		)
-		(property "Intersheetrefs" "${INTERSHEET_REFS}"
-			(at 207.0924 82.55 0)
-			(effects
-				(font
-					(size 1.27 1.27)
-				)
-				(justify left)
-				(hide yes)
-			)
-		)
-	)
-	(global_label "CAN_L"
-		(shape input)
-		(at 198.12 107.95 0)
-		(fields_autoplaced yes)
+	)
+	(hierarchical_label "SDA2"
+		(shape bidirectional)
+		(at 66.04 104.14 0)
 		(effects
 			(font
@@
 			(justify left)
 		)
-		(property "Intersheetrefs" "${INTERSHEET_REFS}"
-			(at 206.79 107.95 0)
-			(effects
-				(font
-					(size 1.27 1.27)
-				)
-				(justify left)
-				(hide yes)
-			)
-		)
-	)
-	(global_label "SDA2"
-		(shape input)
+	)
+	(hierarchical_label "SDA"
+		(shape bidirectional)
 		(at 64.77 81.28 0)
-		(fields_autoplaced yes)
 		(effects
 			(font
@@
 			(justify left)
 		)
-		(property "Intersheetrefs" "${INTERSHEET_REFS}"
-			(at 72.5328 81.28 0)
-			(effects
-				(font
-					(size 1.27 1.27)
-				)
-				(justify left)
-				(hide yes)
-			)
-		)
-	)
-	(global_label "CAN_H"
-		(shape input)
-		(at 132.08 81.28 0)
-		(fields_autoplaced yes)
+	)
+	(hierarchical_label "CAN_H"
+		(shape bidirectional)
+		(at 85.09 36.83 0)
 		(effects
 			(font
@@
 			(justify left)
 		)
-		(property "Intersheetrefs" "${INTERSHEET_REFS}"
-			(at 141.0524 81.28 0)
-			(effects
-				(font
-					(size 1.27 1.27)
-				)
-				(justify left)
-				(hide yes)
-			)
-		)
-	)
-	(global_label "CAN_L"
-		(shape input)
-		(at 198.12 85.09 0)
-		(fields_autoplaced yes)
+	)
+	(hierarchical_label "SCL"
+		(shape bidirectional)
+		(at 64.77 78.74 0)
 		(effects
 			(font
@@
 			(justify left)
 		)
-		(property "Intersheetrefs" "${INTERSHEET_REFS}"
-			(at 206.79 85.09 0)
-			(effects
-				(font
-					(size 1.27 1.27)
-				)
-				(justify left)
-				(hide yes)
-			)
-		)
-	)
-	(global_label "CAN_H"
-		(shape input)
-		(at 85.09 36.83 0)
-		(fields_autoplaced yes)
+	)
+	(hierarchical_label "CAN_L"
+		(shape bidirectional)
+		(at 132.08 83.82 0)
 		(effects
 			(font
@@
 			(justify left)
 		)
-		(property "Intersheetrefs" "${INTERSHEET_REFS}"
-			(at 94.0624 36.83 0)
-			(effects
-				(font
-					(size 1.27 1.27)
-				)
-				(justify left)
-				(hide yes)
-			)
-		)
-	)
-	(global_label "CAN_H"
-		(shape input)
+	)
+	(hierarchical_label "CAN_H"
+		(shape bidirectional)
 		(at 200.66 102.87 0)
-		(fields_autoplaced yes)
 		(effects
 			(font
@@
 			(justify left)
 		)
-		(property "Intersheetrefs" "${INTERSHEET_REFS}"
-			(at 209.6324 102.87 0)
-			(effects
-				(font
-					(size 1.27 1.27)
-				)
-				(justify left)
-				(hide yes)
-			)
-		)
-	)
-	(global_label "SCL2"
-		(shape input)
-		(at 64.77 78.74 0)
-		(fields_autoplaced yes)
+	)
+	(hierarchical_label "CAN_L"
+		(shape bidirectional)
+		(at 198.12 85.09 0)
 		(effects
 			(font
@@
 			(justify left)
 		)
-		(property "Intersheetrefs" "${INTERSHEET_REFS}"
-			(at 72.4723 78.74 0)
-			(effects
-				(font
-					(size 1.27 1.27)
-				)
-				(justify left)
-				(hide yes)
-			)
-		)
-	)
-	(global_label "SDA2"
-		(shape input)
-		(at 66.04 104.14 0)
-		(fields_autoplaced yes)
+	)
+	(hierarchical_label "CAN_H"
+		(shape bidirectional)
+		(at 132.08 81.28 0)
 		(effects
 			(font
@@
 			(justify left)
 		)
-		(property "Intersheetrefs" "${INTERSHEET_REFS}"
-			(at 73.8028 104.14 0)
-			(effects
-				(font
-					(size 1.27 1.27)
-				)
-				(justify left)
-				(hide yes)
-			)
-		)
-	)
-	(global_label "CAN_L"
-		(shape input)
-		(at 132.08 83.82 0)
-		(fields_autoplaced yes)
+	)
+	(hierarchical_label "CAN_L"
+		(shape bidirectional)
+		(at 198.12 107.95 0)
 		(effects
 			(font
@@
 			(justify left)
 		)
-		(property "Intersheetrefs" "${INTERSHEET_REFS}"
-			(at 140.75 83.82 0)
-			(effects
-				(font
-					(size 1.27 1.27)
-				)
-				(justify left)
-				(hide yes)
-			)
-		)
-	)
-	(global_label "CAN_L"
-		(shape input)
+	)
+	(hierarchical_label "CAN_L"
+		(shape bidirectional)
 		(at 85.09 40.64 0)
-		(fields_autoplaced yes)
 		(effects
 			(font
@@
 			(justify left)
 		)
-		(property "Intersheetrefs" "${INTERSHEET_REFS}"
-			(at 93.76 40.64 0)
-			(effects
-				(font
-					(size 1.27 1.27)
-				)
-				(justify left)
-				(hide yes)
-			)
-		)
-	)
-	(global_label "linpot_out"
-		(shape input)
+	)
+	(hierarchical_label "linpot_out"
+		(shape output)
 		(at 132.08 101.6 0)
-		(fields_autoplaced yes)
 		(effects
 			(font
@@
 			(justify left)
 		)
-		(property "Intersheetrefs" "${INTERSHEET_REFS}"
-			(at 144.4992 101.6 0)
-			(effects
-				(font
-					(size 1.27 1.27)
-				)
-				(justify left)
-				(hide yes)
-			)
-		)
-	)
-	(global_label "SCL2"
-		(shape input)
+	)
+	(hierarchical_label "SCL2"
+		(shape bidirectional)
 		(at 66.04 99.06 0)
-		(fields_autoplaced yes)
 		(effects
 			(font
@@
 			)
 			(justify left)
-		)
-		(property "Intersheetrefs" "${INTERSHEET_REFS}"
-			(at 73.7423 99.06 0)
-			(effects
-				(font
-					(size 1.27 1.27)
-				)
-				(justify left)
-				(hide yes)
-			)
 		)
 	)
@@
 			)
 		)
+		(property "P/N" "603-YC324-JK-070RL"
+			(at 171.45 80.01 0)
+			(effects
+				(font
+					(size 1.27 1.27)
+				)
+				(hide yes)
+			)
+		)
 		(pin "8"
 		)
@@
 			)
 		)
+		(property "P/N" "603-YC324-JK-070RL"
+			(at 36.83 96.52 0)
+			(effects
+				(font
+					(size 1.27 1.27)
+				)
+				(hide yes)
+			)
+		)
 		(pin "8"
 		)
@@
 			)
 		)
-		(property "Datasheet" "https://www.yageo.com/upload/media/product/productsearch/datasheet/rchip/PYu-YC_TC_group_51_RoHS_L_9.pdf"
+		(property "Datasheet" "https://www.mouser.com/datasheet/3/508/1/PYu-YC_TC_group_51_RoHS_L_9.pdf"
 			(at 187.96 295.25 0)
 			(effects
@@
 				)
 				(justify left top)
+				(hide yes)
+			)
+		)
+		(property "P/N" "603-YC324-JK-070RL"
+			(at 171.45 100.33 0)
+			(effects
+				(font
+					(size 1.27 1.27)
+				)
 				(hide yes)
 			)
@@
 			)
 		)
+		(property "P/N" "603-YC324-JK-070RL"
+			(at 105.41 78.74 0)
+			(effects
+				(font
+					(size 1.27 1.27)
+				)
+				(hide yes)
+			)
+		)
 		(pin "8"
 		)
@@
 			)
 		)
+		(property "P/N" "603-YC324-JK-070RL"
+			(at 36.83 76.2 0)
+			(effects
+				(font
+					(size 1.27 1.27)
+				)
+				(hide yes)
+			)
+		)
 		(pin "8"
 		)
@@
 				(hide yes)
 			)
+		)
+		(property "P/N" "603-YC324-JK-070RL"
+			(at 105.41 99.06 0)
+			(effects
+				(font
+					(size 1.27 1.27)
+				)
+				(hide yes)
+			)

Commit message: relayout
Parts:
- RN1, RN2, RN4, RN5, RN6, RN7: footprint 4pinRes:YC324JK07220RL -> Air-Sus Footprints:YC324JK07220RL
Connections:
- net +24V: now also RN5.5, RN7.5; no longer RN5.8, RN7.8
- net +3.3V: now also RN1.5; no longer RN1.8
- net CAN_H: now also RN5.6, RN7.6; no longer RN5.7, RN7.7
- net CAN_L: now also RN5.7, RN7.8; no longer RN5.6, RN7.5
- net GND: now also RN1.7, RN5.8, RN7.7; no longer RN1.6, RN5.5, RN7.6
- net Gen_1: now also RN5.4; no longer RN5.1
- net Gen_2: now also RN5.3; no longer RN5.2
- net Gen_3: now also RN5.2; no longer RN5.3
- net Gen_4: now also RN5.1; no longer RN5.4
- net Gen_5: now also RN1.4, RN7.4; no longer RN1.1, RN7.1
- net Gen_6: now also RN1.3, RN7.3; no longer RN1.2, RN7.2
- net Gen_7: now also RN1.2, RN7.2; no longer RN1.3, RN7.3
- net Gen_8: now also RN1.1, RN7.1; no longer RN1.4, RN7.4
- net SCL2: now also RN1.6; no longer RN1.7
- net SDA2: now also RN1.8; no longer RN1.5
