File: hardware/Sus-RH/opamp.kicad_sch (KiCad schematic)
At the start: 5 parts, among them U1 TLV9002QDRQ1

Commit message: layout finished, need to add some more silkscreen + ready for review!
Parts:
- added C2: 1uF, Capacitor_SMD:C_0603_1608Metric_Pad1.08x0.95mm_HandSolder, symbol Device:C
- added R11: 4.7k, Resistor_SMD:R_0603_1608Metric_Pad0.98x0.95mm_HandSolder, symbol Device:R
- R12: value R -> 4.7k; now not fitted
- R13: renamed from R5; value R -> 1k; now not fitted
- R14: renamed from R20; value R -> 0
Connections:
- net GND: now also C2.2
- net linpot_input: now also R11.1; no longer U1.3 (+)
- new net: C2.1, R11.2, U1.3 (+)

Commit message: finished layout + silkscreen, ready to review.
Parts:
- U1: footprint Package_SO:SOIC-8_3.9x4.9mm_P1.27mm -> custom:SOIC8_D_TEX
Changed lines of the file:
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@@
 			)
 		)
-		(property "Footprint" "Package_SO:SOIC-8_3.9x4.9mm_P1.27mm"
+		(property "Footprint" "custom:SOIC8_D_TEX"
 			(at 121.92 29.21 0)
 			(effects
@@
 			)
 		)
-		(property "Footprint" "Package_SO:SOIC-8_3.9x4.9mm_P1.27mm"
+		(property "Footprint" "custom:SOIC8_D_TEX"
 			(at 46.99 43.18 0)
 			(effects
@@
 			)
 		)
-		(property "Footprint" "Package_SO:SOIC-8_3.9x4.9mm_P1.27mm"
+		(property "Footprint" "custom:SOIC8_D_TEX"
 			(at 125.73 60.96 0)
 			(effects
