File: hardware/Sus-RH/opamp.kicad_sch (KiCad schematic)
At the start: 7 parts, among them U1 TLV9002QDRQ1

Commit message: ready to review
Other:
- moved on the sheet: C2
Changed lines of the file:
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@@
 	(wire
 		(pts
+			(xy 99.06 27.94) (xy 99.06 26.67)
+		)
+		(stroke
+			(width 0)
+			(type default)
+		)
+	)
+	(wire
+		(pts
 			(xy 83.82 26.67) (xy 87.63 26.67)
 		)
@@
 	(wire
 		(pts
-			(xy 99.06 34.29) (xy 99.06 35.56)
+			(xy 99.06 35.56) (xy 99.06 36.83)
 		)
 		(stroke
@@
 	(symbol
 		(lib_id "Device:C")
-		(at 99.06 30.48 0)
+		(at 99.06 31.75 0)
 		(unit 1)
 		(exclude_from_sim no)
@@
 		(dnp no)
 		(property "Reference" "C2"
-			(at 102.108 29.21 0)
+			(at 102.108 30.48 0)
 			(effects
 				(font
@@
 		)
 		(property "Value" "1uF"
-			(at 102.108 31.75 0)
+			(at 102.108 33.02 0)
 			(effects
 				(font
@@
 		)
 		(property "Footprint" "Capacitor_SMD:C_0603_1608Metric_Pad1.08x0.95mm_HandSolder"
-			(at 100.0252 34.29 0)
+			(at 100.0252 35.56 0)
 			(effects
 				(font
@@
 		)
 		(property "Datasheet" "~"
-			(at 99.06 30.48 0)
+			(at 99.06 31.75 0)
 			(effects
 				(font
@@
 		)
 		(property "Description" "Unpolarized capacitor"
-			(at 99.06 30.48 0)
+			(at 99.06 31.75 0)
 			(effects
 				(font
@@
 		)
 		(property "Description_1" ""
-			(at 99.06 30.48 0)
+			(at 99.06 31.75 0)
 			(effects
 				(font
@@
 		)
 		(property "Height" ""
-			(at 99.06 30.48 0)
+			(at 99.06 31.75 0)
 			(effects
 				(font
@@
 		)
 		(property "Manufacturer_Name" ""
-			(at 99.06 30.48 0)
+			(at 99.06 31.75 0)
 			(effects
 				(font
@@
 		)
 		(property "Manufacturer_Part_Number" ""
-			(at 99.06 30.48 0)
+			(at 99.06 31.75 0)
 			(effects
 				(font
@@
 		)
 		(property "Mouser Part Number" ""
-			(at 99.06 30.48 0)
+			(at 99.06 31.75 0)
 			(effects
 				(font
@@
 		)
 		(property "Mouser Price/Stock" ""
-			(at 99.06 30.48 0)
+			(at 99.06 31.75 0)
 			(effects
 				(font
@@
 	(symbol
 		(lib_id "power:GND")
-		(at 99.06 35.56 0)
+		(at 99.06 36.83 0)
 		(unit 1)
 		(exclude_from_sim no)
@@
 		(dnp no)
 		(property "Reference" "#PWR028"
-			(at 99.06 41.91 0)
+			(at 99.06 43.18 0)
 			(effects
 				(font
@@
 		)
 		(property "Value" "GND"
-			(at 99.06 39.624 0)
+			(at 99.06 40.894 0)
 			(effects
 				(font
@@
 		)
 		(property "Footprint" ""
-			(at 99.06 35.56 0)
+			(at 99.06 36.83 0)
 			(effects
 				(font
@@
 		)
 		(property "Datasheet" ""
-			(at 99.06 35.56 0)
+			(at 99.06 36.83 0)
 			(effects
 				(font
@@
 		)
 		(property "Description" "Power symbol creates a global label with name \"GND\" , ground"
-			(at 99.06 35.56 0)
+			(at 99.06 36.83 0)
 			(effects
 				(font
