File: hardware/Pitot/diffpress.kicad_sch (KiCad schematic)
At the start: 2 parts, among them IC1 HSCDRRN010NDSA3

Commit message: added layout
Parts:
- IC1: footprint (none) -> UTSVT_Connectors:HSCDRRN010NDSA3
Changed lines of the file:
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@@
 			)
 		)
-		(property "Footprint" ""
+		(property "Footprint" "UTSVT_Connectors:HSCDRRN010NDSA3"
 			(at 132.08 77.47 0)
 			(effects

Commit message: ready to review
Parts:
- IC1: P/N (none) -> HSCDRRN010NDSA3
Other:
- note added: "supposed pull up on spi?? should i just put dnps on here?"
