File: hardware/Pitot/Pitot.kicad_sch (KiCad schematic)
At the start: 28 parts, among them J1 53307-2471, J2 Conn_01x05, J4 Conn_01x08, J5 Conn_01x05, J6 Conn_01x04, J7 Conn_01x04

Commit message: added layout
Parts:
- added F1, F2: 500mA, Fuse:Fuse_0603_1608Metric_Pad1.05x0.95mm_HandSolder, symbol Device:Fuse
- added J3: Conn_01x04, Connector_Molex:Molex_Nano-Fit_105313-xx04_1x04_P2.50mm_Horizontal, symbol Connector_Generic:Conn_01x04
- added J8: Conn_01x02, Connector_PinHeader_2.54mm:PinHeader_1x02_P2.54mm_Vertical, symbol Connector_Generic:Conn_01x02
- J2, J5: footprint (none) -> Connector_Molex:Molex_Nano-Fit_105313-xx05_1x05_P2.50mm_Horizontal
- J6: footprint (none) -> Connector_Molex:Molex_Nano-Fit_105313-xx04_1x04_P2.50mm_Horizontal
- J7: footprint (none) -> Connector_PinHeader_2.54mm:PinHeader_1x04_P2.54mm_Vertical
Connections:
- net +3.3V: now also F1.2, F2.2; no longer J6.1 (Pin_1), J7.1 (Pin_1)
- net Diff1: now also J7.3 (Pin_3)
- net Diff2: now also J8.1 (Pin_1)
- net GND: now also J6.1 (Pin_1), J3.1 (Pin_1), J8.2 (Pin_2); no longer J6.4 (Pin_4)
- net MISO: now also J7.1 (Pin_1)
- net SCL1: now also J6.3 (Pin_3); no longer J6.2 (Pin_2)
- net SCL2: now also J3.3 (Pin_3); no longer J7.2 (Pin_2)
- net SCLK: now also J7.2 (Pin_2)
- net SDA1: now also J6.2 (Pin_2); no longer J6.3 (Pin_3)
- net SDA2: now also J3.2 (Pin_2); no longer J7.3 (Pin_3)
- net pressERR_1: no longer J1.12 (SPI2_NSS)
- net pressERR_2: no longer J1.16 (SPI2_MOSI)
- new net: F1.1, J6.4 (Pin_4)
- new net: F2.1, J3.4 (Pin_4)
Other:
- moved on the sheet: +24v1, +3.3v1, D1, D10, D2, D3, D4, D5, D8, D9, GND1, GND2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

Commit message: ready to review
Parts:
- removed F2: 500mA, Fuse:Fuse_0603_1608Metric_Pad1.05x0.95mm_HandSolder, symbol Device:Fuse
- removed J4: Conn_01x08, Connector_PinHeader_2.54mm:PinHeader_2x04_P2.54mm_Vertical, symbol Connector_Generic:Conn_01x08
- removed J7: Conn_01x04, Connector_PinHeader_2.54mm:PinHeader_1x04_P2.54mm_Vertical, symbol Connector_Generic:Conn_01x04
- removed J8: Conn_01x02, Connector_PinHeader_2.54mm:PinHeader_1x02_P2.54mm_Vertical, symbol Connector_Generic:Conn_01x02
- added J10, J4, J7: Conn_01x03, Connector_PinHeader_2.54mm:PinHeader_1x03_P2.54mm_Vertical, symbol Connector_Generic:Conn_01x03
- added J9: LogicAnalyzer, UTSVT_Connectors:CONN_SFH11-xxxC-D05-ST-XX_SUL, symbol utsvt_connectors:LogicAnalyzer
- added R10, R16, R17, R18, R6, R8, R9: 4.7k, Resistor_SMD:R_0603_1608Metric_Pad0.98x0.95mm_HandSolder, symbol Device:R
- added R11: 4..7k, Resistor_SMD:R_0603_1608Metric_Pad0.98x0.95mm_HandSolder, symbol Device:R
- +24v1, +3.3v1, GND1, GND2: footprint TestPoint:TestPoint_Pad_1.0x1.0mm -> TestPoint:TestPoint_THTPad_2.0x2.0mm_Drill1.0mm
- J2, J5: P/N (none) -> 1053131105
- J3, J6: P/N (none) -> 1053131104
Connections:
- net +3.3V: now also R10.1, R11.1, R16.1, R17.1, R18.1, R6.1, R8.1, R9.1
- net Diff1: now also R11.2
- net Diff2: now also R16.2
- net GND: now also J10.3 (Pin_3), J4.3 (Pin_3), J7.3 (Pin_3), J9.1 (GND)
- net MISO: now also J7.2 (Pin_2), J9.6 (CH4), R17.2
- net P2_LED: now also J1.16 (SPI2_MOSI)
- net SCL1: now also J4.2 (Pin_2), J9.10 (CH0), R6.2
- net SCL2: now also J10.2 (Pin_2), J9.8 (CH2), R9.2
- net SCLK: now also J7.1 (Pin_1), J9.5 (CH5), R18.2
- net SDA1: now also J4.1 (Pin_1), J9.9 (CH1), R8.2
- net SDA2: now also J10.1 (Pin_1), J9.7 (CH3), R10.2
- net fused_3.3v: now reaches F1.1, J6.4 (Pin_4)
- net fused_3.3v: now also J3.4 (Pin_4)
- net CAN_+ renamed CAN_H
- net CAN_- renamed CAN_L
- no-connect marks 1 -> 4
Other:
- moved on the sheet: J1, J2, J3, J5, J6, R4, R5

Commit message: finished pitot board
Parts:
- removed J10, J4, J7: Conn_01x03, Connector_PinHeader_2.54mm:PinHeader_1x03_P2.54mm_Vertical, symbol Connector_Generic:Conn_01x03
- +24v1, +3.3v1, GND1, GND2: now left out of the parts list
- R10, R16, R6, R8, R9: value 4.7k -> 10k; P/N (none) -> CRCW060310K0FKEI
- R11: value 4..7k -> 10k; P/N (none) -> CRCW060310K0FKEI
- R17, R18: P/N (none) -> CRCW06034K70FKEA
Connections:
- net +3.3V: no longer R7.1
- net Diff1: now also J9.4 (CH6)
- net Diff2: now also J9.3 (CH7)
- net at R7.2: no longer D2.2 (A)
- no-connect marks 4 -> 2
Other:
- moved on the sheet: R11, R7, R8, R9

Commit message: pitot board ordered, routing+size finished for temperature board so pull??
Connections:
- net +3.3V: now also R7.1
- net at R7.2: now also D2.2 (A)
Other:
- moved on the sheet: R7
Changed lines of the file:
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@@
 	(symbol
 		(lib_id "Device:R")
-		(at 30.48 88.9 0)
+		(at 29.21 88.9 0)
 		(unit 1)
 		(exclude_from_sim no)
@@
 		(dnp no)
 		(property "Reference" "R7"
-			(at 32.258 87.63 0)
+			(at 30.988 87.63 0)
 			(effects
 				(font
@@
 		)
 		(property "Value" "120"
-			(at 32.512 89.9161 0)
+			(at 31.242 89.9161 0)
 			(effects
 				(font
@@
 		)
 		(property "Footprint" "Resistor_SMD:R_0603_1608Metric_Pad0.98x0.95mm_HandSolder"
-			(at 28.702 88.9 90)
+			(at 27.432 88.9 90)
 			(effects
 				(font
@@
 		)
 		(property "Datasheet" "~"
-			(at 30.48 88.9 0)
+			(at 29.21 88.9 0)
 			(effects
 				(font
@@
 		)
 		(property "Description" "Resistor"
-			(at 30.48 88.9 0)
+			(at 29.21 88.9 0)
 			(effects
 				(font
@@
 		)
 		(property "P/N" "CRCW06031K00FKEI "
-			(at 30.48 88.9 0)
+			(at 29.21 88.9 0)
 			(effects
 				(font
@@
 		)
 		(property "JLC P/N" ""
-			(at 30.48 88.9 0)
+			(at 29.21 88.9 0)
 			(effects
 				(font
