File: hardware/ir_board/ir_board.kicad_pcb (KiCad board)
At the start: 2 copper layers, 25.2 x 30 mm, 22 parts, among them J1 Conn_01x04, J2 Conn_01x06, Q1 IRLML0030, U1 VL53L0CXV0DH1

Commit message: fixed drc and made gerbers
Routing:
- net /GPIO1: track 48.4 -> 51.8 mm
- net /SDA: track 34.6 -> 35.3 mm, vias 0 -> 1
- net /SCL: track 30.9 -> 31.0 mm, vias 0 -> 1
Other:
- board text added: "3.3V"
Changed lines of the file:
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@@
 			(psa4output no)
 			(plot_black_and_white yes)
+			(plotinvisibletext no)
 			(sketchpadsonfab no)
 			(plotpadnumbers no)
@@
 		)
 	)
+	(gr_text "3.3V"
+		(at 167.5 59.8 0)
+		(layer "B.SilkS")
+		(effects
+			(font
+				(size 1 1)
+				(thickness 0.15)
+			)
+			(justify mirror)
+		)
+	)
 	(segment
 		(start 159.95 68.5)
@@
 	)
 	(segment
-		(start 156.2 75.05)
+		(start 156.75 75.6)
+		(end 158.275 75.6)
+		(width 0.5)
+		(layer "F.Cu")
+		(net 5)
+	)
+	(segment
+		(start 155.65 74.5)
 		(end 156.75 75.6)
 		(width 0.5)
@@
 	)
 	(segment
-		(start 156.75 75.6)
-		(end 158.275 75.6)
+		(start 155.65 74.1)
+		(end 155.65 74.5)
 		(width 0.5)
 		(layer "F.Cu")
@@
 	)
 	(via
-		(at 156.2 75.05)
+		(at 155.65 74.1)
 		(size 0.6)
 		(drill 0.3)
@@
 	)
 	(segment
-		(start 155.65 74.5)
-		(end 155.65 69.5)
-		(width 0.5)
-		(layer "B.Cu")
-		(net 5)
-	)
-	(segment
 		(start 155.75 69.6)
 		(end 155.65 69.5)
@@
 	)
 	(segment
-		(start 156.2 75.05)
-		(end 155.65 74.5)
+		(start 155.65 74.1)
+		(end 155.65 69.5)
 		(width 0.5)
 		(layer "B.Cu")
@@
 	)
 	(segment
-		(start 162.3 76.525)
-		(end 162.25 76.475)
-		(width 0.2)
-		(layer "F.Cu")
-		(net 6)
-	)
-	(segment
-		(start 163.125 76.487068)
-		(end 163.087068 76.525)
+		(start 162.3 77.5)
+		(end 162.3 76.525)
 		(width 0.2)
 		(layer "F.Cu")
@@
 	)
 	(segment
-		(start 163.087068 76.525)
-		(end 162.3 76.525)
+		(start 158.35 59.15)
+		(end 159.2 60)
 		(width 0.2)
 		(layer "F.Cu")
@@
 	)
 	(segment
-		(start 158.35 59.15)
-		(end 159.2 60)
+		(start 162.3 76.525)
+		(end 162.25 76.475)
 		(width 0.2)
 		(layer "F.Cu")
@@
 	)
 	(via
-		(at 163.125 76.487068)
+		(at 162.3 77.5)
 		(size 0.6)
 		(drill 0.3)
@@
 	)
 	(segment
-		(start 167 71.62)
-		(end 170.45 68.17)
-		(width 0.2)
-		(layer "B.Cu")
-		(net 6)
-	)
-	(segment
 		(start 158.75 56.25)
 		(end 158.75 59.75)
@@
 	)
 	(segment
-		(start 170.45 68.17)
-		(end 172.7 65.92)
+		(start 167.149361 77.8)
+		(end 167.849 77.100361)
 		(width 0.2)
 		(layer "B.Cu")
@@
 	)
 	(segment
-		(start 163.125 76.487068)
-		(end 165.462932 76.487068)
+		(start 167.849 70.771)
+		(end 170.45 68.17)
 		(width 0.2)
 		(layer "B.Cu")
@@
 	)
 	(segment
-		(start 171.626694 55.118152)
-		(end 171.142554 54.885003)
+		(start 162.6 77.8)
+		(end 167.149361 77.8)
 		(width 0.2)
 		(layer "B.Cu")
@@
 	)
 	(segment
-		(start 172.7 56.729868)
-		(end 172.614997 56.357446)
+		(start 162.3 77.5)
+		(end 162.6 77.8)
+		(width 0.2)
+		(layer "B.Cu")
+		(net 6)
+	)
+	(segment
+		(start 170.45 68.17)
+		(end 172.7 65.92)
 		(width 0.2)
 		(layer "B.Cu")
@@
 	)
 	(segment
-		(start 165.462932 76.487068)
-		(end 167 74.95)
+		(start 171.626694 55.118152)
+		(end 171.142554 54.885003)
+		(width 0.2)
+		(layer "B.Cu")
+		(net 6)
+	)
+	(segment
+		(start 172.7 56.729868)
+		(end 172.614997 56.357446)
 		(width 0.2)
 		(layer "B.Cu")
@@
 	)
 	(segment
-		(start 167 74.95)
-		(end 167 71.62)
+		(start 167.849 77.100361)
+		(end 167.849 70.771)
 		(width 0.2)
 		(layer "B.Cu")
@@
 	)
 	(segment
+		(start 161.8 64.7)
+		(end 161.8 65.425)
+		(width 0.2)
+		(layer "F.Cu")
+		(net 7)
+	)
+	(segment
 		(start 172.25 61.29)
 		(end 172.25 56.3)
@@
 	)
 	(segment
-		(start 162.401 64.874)
-		(end 161.825 65.45)
-		(width 0.2)
-		(layer "F.Cu")
-		(net 7)
-	)
-	(segment
-		(start 162.401 60.901)
-		(end 162.401 64.874)
+		(start 161.25 56.25)
+		(end 161.25 59.75)
 		(width 0.2)
 		(layer "F.Cu")
@@
 	)
 	(segment
-		(start 161.25 56.25)
-		(end 161.25 59.75)
+		(start 162.35 55.15)
+		(end 161.25 56.25)
 		(width 0.2)
 		(layer "F.Cu")
@@
 	)
 	(segment
-		(start 162.35 55.15)
-		(end 161.25 56.25)
+		(start 161.8 65.425)
+		(end 161.825 65.45)
 		(width 0.2)
 		(layer "F.Cu")
@@
 		(net 7)
 	)
+	(via
+		(at 161.8 64.7)
+		(size 0.6)
+		(drill 0.3)
+		(layers "F.Cu" "B.Cu")
+		(net 7)
+	)
 	(segment
 		(start 161.25 59.75)
 		(end 162.401 60.901)
 		(width 0.2)
-		(layer "F.Cu")
+		(layer "B.Cu")
+		(net 7)
+	)
+	(segment
+		(start 162.401 60.901)
+		(end 162.401 64.099)
+		(width 0.2)
+		(layer "B.Cu")
+		(net 7)
+	)
+	(segment
+		(start 162.401 64.099)
+		(end 161.8 64.7)
+		(width 0.2)
+		(layer "B.Cu")
 		(net 7)
 	)
 	(segment
-		(start 160.3125 63.8125)
+		(start 160.1625 65.6)
 		(end 160.3125 65.45)
 		(width 0.2)
@@
 	)
 	(segment
+		(start 159.5 65.6)
+		(end 160.1625 65.6)
+		(width 0.2)
+		(layer "F.Cu")
+		(net 8)
+	)
+	(segment
 		(start 160.3125 65.45)
 		(end 160.3 65.4625)
@@
 		(net 8)
 	)
+	(via
+		(at 159.5 65.6)
+		(size 0.6)
+		(drill 0.3)
+		(layers "F.Cu" "B.Cu")
+		(net 8)
+	)
 	(segment
-		(start 158.75 62.25)
-		(end 160.3125 63.8125)
+		(start 159.5 63)
+		(end 159.5 65.6)
 		(width 0.2)
-		(layer "F.Cu")
+		(layer "B.Cu")
 		(net 8)
 	)
@@
 		(width 0.2)
 		(layer "B.Cu")
+		(net 8)
+	)
+	(segment
+		(start 158.75 62.25)
+		(end 159.5 63)
+		(width 0.2)
+		(layer "B.Cu")

Commit message: pitot board ordered, routing+size finished for temperature board so pull??
Parts:
- removed G***: LHRs_LOGO, UTSVT_Logos:LHRs_LOGO
- added +3.3v: TestPoint, TestPoint:TestPoint_THTPad_1.5x1.5mm_Drill0.7mm, F.Cu at (155.5, 56.8)
- added GND: TestPoint, TestPoint:TestPoint_THTPad_1.5x1.5mm_Drill0.7mm, F.Cu at (167.0, 57.2)
- C1: value 10uf -> 4.7uf; footprint Capacitor_SMD:C_0603_1608Metric_Pad1.08x0.95mm_HandSolder -> Capacitor_SMD:C_0805_2012Metric_Pad1.18x1.45mm_HandSolder
- J1: value Conn_01x04 -> Conn_01x05; footprint Connector_PinHeader_2.54mm:PinHeader_1x04_P2.54mm_Vertical -> Connector_PinSocket_2.54mm:PinSocket_1x05_P2.54mm_Vertical; moved to F.Cu
- moved J1 2.75 mm to (170.5, 60.3), turned to 0 degrees
- moved C1 0.30 mm to (166.0, 67.8)
Connections:
- J1 pad 1: /SCL -> +3.3V
- J1 pad 2: /SDA -> /SCL
- J1 pad 3: /GPIO1 -> /SDA
- J1 pad 4: GND -> /GPIO1
Routing:
- net /SDA: track 35.3 -> 34.6 mm
- net +3.3V: track 14.0 -> 14.4 mm, vias 8 -> 7
Other:
- board text added: "+3.3V"
- board text added: "GND"
- board text added: "INT"
- board text added: "Karthik Kurapati Rev B Febuary 2026"
- board text added: "Rideheight Breakout"
- board text added: "SCL"
- board text added: "SDA"
- board text removed: "3.3V"
