File: hardware/ir_board/ir_board.kicad_sch (KiCad schematic)
At the start: 23 parts, among them J1 Conn_01x04, J2 Conn_01x06, Q1 IRLML0030, U1 VL53L0CXV0DH1

Commit message: pitot board ordered, routing+size finished for temperature board so pull??
Parts:
- removed J1: Conn_01x04, Connector_PinHeader_2.54mm:PinHeader_1x04_P2.54mm_Vertical, symbol Connector_Generic:Conn_01x04
- removed TP1, TP2: TestPoint, symbol Connector:TestPoint
- added +3.3vTP1, GNDTP2: TestPoint, TestPoint:TestPoint_THTPad_1.5x1.5mm_Drill0.7mm, symbol Connector:TestPoint
- added J1: Conn_01x05, Connector_PinSocket_2.54mm:PinSocket_1x05_P2.54mm_Vertical, symbol Connector_Generic:Conn_01x05
- C1: value 10uf -> 4.7uf; footprint Capacitor_SMD:C_0603_1608Metric_Pad1.08x0.95mm_HandSolder -> Capacitor_SMD:C_0805_2012Metric_Pad1.18x1.45mm_HandSolder; P/N GRM21BR61H106KE43K -> MLASH168SB7104KTNA01
Connections:
- net +3.3V: now also +3.3vTP1.1, J1.1 (Pin_1)
- net GND: now also GNDTP2.1, J1.5 (Pin_5)
- net GPIO1: now also J1.4 (Pin_4)
- net SCL: now also J1.2 (Pin_2)
- net SDA: now also J1.3 (Pin_3)
- no-connect marks 3 -> 1
Other:
- note removed: "Nano-fit"
